Commit message: Audit, fix, and harden entire codebase for hardware readiness
Critical fixes found by full audit:
- URDF wheel radius (0.15->0.075) and separation (0.45->0.40) mismatched
  every other config — robot would have driven in circles
- All launch file executable names wrong (didn't match setup.py entry points)
- Non-existent safety_monitor_node replaced with actual 5 safety nodes
- 3 nodes missing from launch files (odom_publisher, datum_setter, speed_regulator)
- Odom topic mismatch (wheel_odom vs odom/wheel) broke EKF fusion
- Nav2 robot radius too small (0.25->0.36) — would cause collisions
- Safety supervisor never subscribed to obstacle distance
- Ultrasonic frame_ids didn't match URDF link names
- Fake GPS parameter name mismatch (noise_stddev vs noise_std_m)
- Speed regulator max speed inconsistent with Nav2 config (1.5->1.0)

New features:
- Real rclpy mode in ros_bridge.py (subscribers, publishers, service
  clients, threaded spin, asyncio bridge, auto-reconnection)
- NTRIP client node for RTK GPS corrections (rtk2go.com compatible)
- GPS node now accepts binary RTCM corrections from NTRIP client

Documentation:
- docs/topic_map.md — full system wiring diagram (all topics/services/TFs)
- docs/wiring_guide.md — pin assignments, power budget, safety circuit,
  32-step assembly checklist
- docs/bom.md — 67-item BOM with part numbers, ~$1,357 total

Project config:
- pyproject.toml (pytest, ruff config)
- Top-level requirements.txt (all Python deps)

Co-Authored-By: Claude Opus 4.6 <noreply@anthropic.com>

File: striper_ws/src/striper_description/urdf/striper.urdf.xacro (robot description, xacro)
@@ -6,8 +6,8 @@
   <xacro:property name="chassis_height" value="0.15"/>
   <xacro:property name="chassis_mass"   value="15.0"/>
-  <xacro:property name="wheel_radius" value="0.15"/>
+  <xacro:property name="wheel_radius" value="0.075"/>
   <xacro:property name="wheel_width"  value="0.05"/>
   <xacro:property name="wheel_mass"   value="1.0"/>
-  <xacro:property name="wheel_separation" value="0.45"/>
+  <xacro:property name="wheel_separation" value="0.40"/>
   <xacro:property name="caster_radius" value="0.05"/>
   <xacro:property name="caster_mass"   value="0.3"/>
@@ -128,5 +128,5 @@
     <parent link="base_link"/>
     <child link="caster_wheel"/>
-    <origin xyz="${-chassis_length/2 + caster_radius} 0 ${caster_radius}" rpy="0 0 0"/>
+    <origin xyz="${-chassis_length/2 + caster_radius} 0 ${-(wheel_radius - caster_radius)}" rpy="0 0 0"/>
   </joint>
   <gazebo reference="caster_wheel">
